File: CRBN 60.sch (EAGLE design)
At the start: 148 parts, among them IC3 HOLYIOT_18010, IC4 FS312F-G, Q4 FS8205, Q5 PMOSFET, Q6 PMOSFET, U2 AP2112K-3.3TRG1

Commit message: tweaks and checks
Parts:
- removed Q6: PMOSFET, Transistor:PMOSFET_SOT23
- removed R18: 2k, rcl:R-EU_R0603
- added J1: (no value), SparkFun-Connectors:CONN_051.27MM
- added LED1: (no value), led:LEDSML0603
- added R1: 1k, rcl:R-EU_R0603
- added R2: 10k, rcl:R-EU_R0603
- added S1: MOMENTARY-SWITCH-SPST-SMD-6.2MM-TALL, SparkFun-Switches:MOMENTARY-SWITCH-SPST-SMD-6.2MM-TALL
Connections:
- removed net LED_VCC: Q6.S
- new net N$17: IC3.P1.07, J1.1
- new net N$2: LED1.C, R1.2
- new net N$32: IC3.P1.05, J1.2
- new net N$46: IC3.P0.24, J1.3
- new net N$59: IC3.P0.20, J1.4
- new net N$67: IC3.P0.17, J1.5
- net BLED: now also LED1.A
- net GND: now also R1.1, S1.2; no longer R18.2
- net POWER_PIN: no longer Q6.G, R18.1
- net RESET: now also R2.2, S1.1
- net VDD_NRF: now also R2.1; no longer Q6.D
