File: CRBN 60.brd (EAGLE design)
At the start: 295.3 x 104.8 mm, 148 parts, among them IC3 HOLYIOT_18010, IC4 FS312F-G, Q4 FS8205, Q5 PMOSFET, Q6 PMOSFET, U2 AP2112K-3.3TRG1

Commit message: tweaks and checks
Parts:
- removed Q6: PMOSFET, Transistor:SOT23
- removed R18: 2k, rcl:R0603
- added J1: (no value), SparkFun-Connectors:1X05_1.27MM
- added LED1: (no value), led:SML0603
- added R1: 1k, rcl:R0603
- added R2: 10k, rcl:R0603
- added S1: MOMENTARY-SWITCH-SPST-SMD-6.2MM-TALL, SparkFun-Switches:TACTILE_SWITCH_SMD_6.2MM_TALL
Connections:
- removed net LED_VCC: Q6.2
- new net N$17: IC3.P1.07, J1.1
- new net N$2: LED1.C, R1.2
- new net N$32: IC3.P1.05, J1.2
- new net N$46: IC3.P0.24, J1.3
- new net N$59: IC3.P0.20, J1.4
- new net N$67: IC3.P0.17, J1.5
- net BLED: now also LED1.A
- net GND: now also R1.1, S1.B2; no longer R18.2
- net POWER_PIN: no longer Q6.1, R18.1
- net RESET: now also R2.2, S1.A2
- net VDD_NRF: now also R2.1; no longer Q6.3
Routing:
- net POWER_PIN: track 17.9 -> 0.01 mm, vias 2 -> 0
- net N$67: track 0.00 -> 17.2 mm
- net N$59: track 0.00 -> 14.6 mm
- net BLED: track 0.00 -> 12.2 mm, vias 0 -> 2
- net N$46: track 0.00 -> 12.0 mm
- net N$32: track 0.00 -> 9.37 mm
- net N$17: track 0.00 -> 6.78 mm
- net VDD_NRF: track 59.7 -> 63.7 mm
- net RESET: track 109.1 -> 112.8 mm, vias 5 -> 6
- net N$2: track 0.00 -> 2.08 mm
- net GND: track 55.6 -> 57.2 mm
- net V_USB: track 288.4 -> 287.7 mm

Commit message: new board
Routing:
- net RESET: track 112.8 -> 250.1 mm
- net GND: track 57.2 -> 159.9 mm
- net ROW3: track 512.9 -> 540.8 mm
- net ROW2: track 538.3 -> 566.2 mm
- net ROW1: track 563.2 -> 591.2 mm
- net BVOLT: track 15.0 -> 42.9 mm
- net COL1: track 177.7 -> 205.6 mm
- net ROW4: track 485.1 -> 513.0 mm
- net POWER_PIN: track 0.01 -> 28.0 mm
- net COL4: track 93.9 -> 121.9 mm
- net N$59: track 14.6 -> 42.5 mm
- net N$67: track 17.2 -> 45.1 mm
- net COL5: track 100.4 -> 128.3 mm
- net ROW5: track 472.8 -> 500.8 mm
- net COL2: track 169.0 -> 196.9 mm
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