File: CRBN-60-soldered.brd (EAGLE design)
At the start: 285.8 x 94.6 mm, 206 parts, among them CN2 BM02B-SRSS-TB, IC3 HOLYIOT_18010, IC4 FS312F-G, Q4 FS8205, Q5 PMOSFET, U2 AP2112K-3.3TRG1, X5U_1 CHERRY-SOLDER, X5U_2 CHERRY-SOLDER

Commit message: updates
Parts:
- U$66: value 2.5MM_HOLE -> 2.5MM_ELONGATED; device Volume_V1:2.5MM_HOLE -> Volume_V1:2.5MM_ELONGATED
- moved J4 30.1 mm to (144.2, 80.1)
- moved CN2 29.5 mm to (142.9, 87.0)
Routing:
- net G_BAT: track 78.6 -> 124.0 mm, vias 2 -> 3
- net V_BATT: track 79.5 -> 122.4 mm
- net ROW2: vias 2 -> 4
- net ROW1: vias 2 -> 4
- net GND: vias 12 -> 13
