File: CRBN-60-soldered.brd (EAGLE design)
At the start: 285.8 x 94.6 mm, 206 parts, among them CN2 BM02B-SRSS-TB, IC3 HOLYIOT_18010, IC4 FS312F-G, Q4 FS8205, Q5 PMOSFET, U2 AP2112K-3.3TRG1, X5U_1 CHERRY-SOLDER, X5U_2 CHERRY-SOLDER

Commit message: updatyes
Parts:
- removed IC4: FS312F-G, FS312F-G:SOT95P280X145-6N
- removed Q4: FS8205, FS8205:FS8205
- removed R16: 2k, rcl:R0603
- removed U$63: TP4056, TP4056:SOT23-8
- added D69, D70, D71, D72, D73, D74, D75, D76: 1N4148WS, Diodes:SOD-323
- added FUSE: 500m, rcl:R0603
- added J1: (no value), SparkFun-Connectors:1X04_NO_SILK
- added U$3: XB3303ASOT23, Volume_V1:SOT23-3
- added U$4: TP4056SOI8, TP4056:SOIC8
- PROG1: device SparkFun-Connectors:1X06_HOLES_ONLY -> SparkFun-Connectors:1X06_NO_SILK
- moved IC3 35.6 mm to (89.1, 16.9)
- moved R2 16.7 mm to (156.1, 10.3)
- moved R_SHIFT_1.75U_RIGHT 2.38 mm to (259.6, 33.3)
- moved CN2 2.14 mm to (143.7, 85.0), turned to 90 degrees
- moved J4 1.85 mm to (142.4, 79.6)
- moved C6 0.72 mm to (102.9, 10.2)
- moved R20 0.43 mm to (105.7, 9.53)
- moved C4 0.33 mm to (102.6, 20.9)
- moved Q5 0.15 mm to (113.5, 20.8)
- moved R14 0.08 mm to (102.5, 18.1)
- flipped LED1 to the bottom
- flipped LED2 to the bottom
Connections:
- removed net N$77: IC4.1, Q4.4
- removed net N$78: IC4.3, Q4.6
- removed net N$79: C5.1, IC4.5, R15.1
- removed net N$80: IC4.2, R16.2
- new net N$50: C5.1, R15.1, U$3.2
- new net N$67: FUSE.2, J3.VBUS1, J3.VBUS2
- net D+: now also D69.C, J1.2
- net D-: now also D70.C, J1.3
- net GND: now also D69.A, D70.A, D71.A, D72.A, J1.1, U$3.1, U$4.1, U$4.3, U$64.P$1, U$64.P$2, U$65.P$1, U$65.P$2, U$66.P$1, U$66.P$2, U$67.P$1, U$67.P$2; no longer Q4.1, R16.1, U$63.1, U$63.3
- net G_BAT: now also U$3.3; no longer IC4.6, Q4.3
- net N$74: now also U$4.2; no longer U$63.2
- net N$76: now also U$4.7; no longer U$63.7
- net VDD_NRF: now also D72.C
- net V_BATT: now also U$4.5; no longer U$63.5
- net V_USB: now also D71.C, FUSE.1, J1.4, U$4.4, U$4.8; no longer J3.VBUS1, J3.VBUS2, U$63.4, U$63.8
Routing:
- net V_USB: track 330.2 -> 396.9 mm, vias 10 -> 11
- net D-: track 200.7 -> 248.9 mm, vias 4 -> 7
- net N$18: track 8.85 -> 33.5 mm, vias 0 -> 1
- net D+: track 202.0 -> 226.5 mm, vias 4 -> 6
- net N$52: track 11.9 -> 32.7 mm, vias 0 -> 1
- net N$67: track 0.00 -> 16.8 mm, vias 0 -> 2
- net N$76: track 8.08 -> 22.6 mm, vias 0 -> 4
- net RESET: track 180.0 -> 194.5 mm, vias 6 -> 7
- net VDD_NRF: track 76.6 -> 90.8 mm, vias 3 -> 5
- net COL15: track 290.7 -> 304.6 mm, vias 3 -> 5
- net COL14: track 319.6 -> 329.6 mm, vias 3 -> 5
- net N$78: track 9.33 -> 0.00 mm, vias 2 -> 0
- net N$79: track 8.60 -> 0.00 mm
- net N$50: track 0.00 -> 7.98 mm
- net G_BAT: track 124.0 -> 130.0 mm
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Other:
- board size 285.8 x 94.6 mm -> 283.8 x 94.6 mm
- board text added: "+"
- board text added: "D+"
- board text added: "D-"
- board text added: "SPARES"
- board text removed: "+ -"
- board text removed: "POLARITY WORKS 60"
