File: CRBN-60-soldered.sch (EAGLE design)
At the start: 206 parts, among them CN2 BM02B-SRSS-TB, IC3 HOLYIOT_18010, IC4 FS312F-G, Q4 FS8205, Q5 PMOSFET, U2 AP2112K-3.3TRG1, X5U_1 CHERRY-SOLDER, X5U_2 CHERRY-SOLDER

Commit message: updates
Parts:
- U$66: value 2.5MM_HOLE -> 2.5MM_ELONGATED; device Volume_V1:2.5MM_HOLE -> Volume_V1:2.5MM_ELONGATED
Changed lines of the file:
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@@
 <part name="U$65" library="Volume_V1" deviceset="2.5MM_ELONGATED" device=""/>
 <part name="U$67" library="Volume_V1" deviceset="2.5MM_ELONGATED" device=""/>
-<part name="U$66" library="Volume_V1" deviceset="2.5MM_HOLE" device=""/>
+<part name="U$66" library="Volume_V1" deviceset="2.5MM_ELONGATED" device=""/>
 <part name="U$62" library="Volume_V1" deviceset="SMD-BUTTON" device=""/>
 <part name="U$68" library="Volume_V1" deviceset="STAB-2U" device=""/>

Commit message: updatyes
Parts:
- removed IC4: FS312F-G, FS312F-G:FS312F-G
- removed Q4: FS8205, FS8205:FS8205
- removed R16: 2k, rcl:R-EU_R0603
- removed U$63: TP4056, TP4056:TP4056
- added D69, D70, D71, D72, D73, D74, D75, D76: 1N4148WS, Diodes:1N4148WS
- added FUSE: 500m, rcl:R-EU_R0603
- added J1: (no value), SparkFun-Connectors:CONN_041X04_NO_SILK
- added U$3: XB3303ASOT23, Volume_V1:XB3303ASOT23
- added U$4: TP4056SOI8, TP4056:TP4056SOI8
- PROG1: device SparkFun-Connectors:CONN_06POGOPIN_HOLES_ONLY -> SparkFun-Connectors:CONN_06NO_SILK_FEMALE_PTH
Connections:
- removed net N$77: IC4.OD, Q4.G2
- removed net N$78: IC4.OC, Q4.G1
- removed net N$79: C5.1, IC4.VCC, R15.1
- removed net N$80: IC4.CS, R16.2
- new net N$50: C5.1, R15.1, U$3.VDD
- new net N$67: FUSE.2, J3.VBUS
- net D+: now also D69.C, J1.2
- net D-: now also D70.C, J1.3
- net GND: now also D69.A, D70.A, D71.A, D72.A, J1.1, U$3.VM, U$4.GND, U$4.TEMP, U$64.P$1, U$65.P$1, U$66.P$1, U$67.P$1; no longer Q4.S1, R16.1, U$63.GND, U$63.TEMP
- net G_BAT: now also U$3.GND; no longer IC4.GND, Q4.S2
- net N$74: now also U$4.PROG; no longer U$63.PROG
- net N$76: now also U$4.!CHRG; no longer U$63.!CHRG
- net VDD_NRF: now also D72.C
- net V_BATT: now also U$4.BAT; no longer U$63.BAT
- net V_USB: now also D71.C, FUSE.1, J1.4, U$4.CE, U$4.VCC; no longer J3.VBUS, U$63.CE, U$63.VCC
Other:
- moved on the sheet: C5
