File: CRBN-60.brd (EAGLE design)
At the start: 285.8 x 94.6 mm, 160 parts, among them IC3 HOLYIOT_18010, IC4 FS312F-G, Q4 FS8205, Q5 PMOSFET, U2 AP2112K-3.3TRG1

Commit message: library updates
Parts:
- U$63: value TP4056 -> TP4056SOI8; device TP4056:SOT23-8 -> TP4056:SOIC8
Routing:
- net RESET: track 195.2 -> 199.1 mm
Changed lines of the file:
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@@
 </layers>
 <board>
-<fusionsync huburn="a.cGVyc29uYWw6dWUyZjhiMzhi" projecturn="a.cGVyc29uYWw6dWUyZjhiMzhiIzIwMjAxMDEwMzQxNDg0MzAx" f3durn="urn:adsk.wipprod:dm.lineage:ftLnUbcxSgCAcFjv9yPAJg" pcbguid="" lastpulledtime="" lastsyncedchangeguid="" latestrevisionid="" lastsyncedrevisionid="" lastboardhashguid="" lastpushedtime="" linktopcb3d="false"/>
+<fusionsync huburn="a.cGVyc29uYWw6dWUyZjhiMzhi" projecturn="a.cGVyc29uYWw6dWUyZjhiMzhiIzIwMjAxMDEwMzQxNDg0MzAx" f3durn="urn:adsk.wipprod:dm.lineage:ftLnUbcxSgCAcFjv9yPAJg" pcbguid="" lastpulledtime="" lastsyncedchangeguid="" latestrevisionid="" lastsyncedrevisionid="" lastboardhashguid="" lastpushedtime="" linktopcb3d="true"/>
 <plain>
 <text x="138.0998" y="12.75715" size="1.27" layer="26" rot="MR90">VREF</text>
@@
 <attribute name="NAME" x="102.2858" y="22.0218" size="0.6096" layer="26" rot="MR180"/>
 </element>
-<element name="U$63" library="TP4056" package="SOT23-8" value="TP4056" x="106.16565" y="18.86585" smashed="yes" rot="MR90">
+<element name="U$63" library="TP4056" package="SOIC8" value="TP4056SOI8" x="106.16565" y="18.86585" smashed="yes" rot="MR90">
 <attribute name="NAME" x="107.18185" y="19.75485" size="0.6096" layer="26" ratio="10" rot="MR0"/>
 </element>
@@
 <wire x1="101.558" y1="12.57935" x2="102.4754" y2="10.09015" width="0" layer="19" extent="16-16"/>
 <wire x1="100.81985" y1="15.3924" x2="100.4824" y2="13.208" width="0" layer="19" extent="16-16"/>
-<wire x1="103.58565" y1="16.96085" x2="100.81985" y2="15.72138125" width="0" layer="19" extent="16-16"/>
-<wire x1="102.1588" y1="19.0382" x2="103.58565" y2="16.96085" width="0" layer="19" extent="16-16"/>
-<wire x1="103.58565" y1="19.50085" x2="102.1588" y2="19.0382" width="0" layer="19" extent="16-16"/>
+<wire x1="103.41565" y1="16.96085" x2="100.81985" y2="15.72138125" width="0" layer="19" extent="16-16"/>
+<wire x1="102.1588" y1="19.0382" x2="103.41565" y2="16.96085" width="0" layer="19" extent="16-16"/>
+<wire x1="103.41565" y1="19.50085" x2="102.1588" y2="19.0382" width="0" layer="19" extent="16-16"/>
 <wire x1="95.677353125" y1="10.54055" x2="100.4824" y2="13.208" width="0" layer="19" extent="16-16"/>
 <wire x1="82.477353125" y1="10.54055" x2="83.312" y2="12.7508" width="0" layer="19" extent="16-16"/>
@@
 <wire x1="23.84425" y1="40.3225" x2="23.84425" y2="25.0825" width="0" layer="19" extent="16-16"/>
 <wire x1="23.84425" y1="40.3225" x2="23.84425" y2="40.3225" width="0" layer="19" extent="1-16"/>
-<wire x1="22.9898" y1="54.7414" x2="23.84425" y2="40.3225" width="0" layer="19" extent="16-16"/>
-<wire x1="16.9898" y1="54.7414" x2="22.9898" y2="54.7414" width="0" layer="19" extent="16-16"/>
-<wire x1="16.0528" y1="71.7804" x2="16.9898" y2="54.7414" width="0" layer="19" extent="16-16"/>
+<wire x1="24.6898" y1="55.1164" x2="23.84425" y2="40.3225" width="0" layer="19" extent="16-16"/>
+<wire x1="15.2898" y1="55.1164" x2="24.6898" y2="55.1164" width="0" layer="19" extent="16-16"/>
+<wire x1="16.0528" y1="71.7804" x2="15.2898" y2="55.1164" width="0" layer="19" extent="16-16"/>
 <wire x1="16.0528" y1="71.7804" x2="16.0528" y2="71.7804" width="0" layer="19" extent="1-16"/>
-<wire x1="-0.03175" y1="40.3225" x2="16.9898" y2="54.7414" width="0" layer="19" extent="16-16"/>
+<wire x1="-0.03175" y1="40.3225" x2="15.2898" y2="55.1164" width="0" layer="19" extent="16-16"/>
 <wire x1="-0.03175" y1="40.3225" x2="-0.03175" y2="40.3225" width="0" layer="19" extent="1-16"/>
 <wire x1="-0.0254" y1="28.829" x2="-0.03175" y2="40.3225" width="0" layer="19" extent="16-16"/>
@@
 <wire x1="4.826" y1="92.202" x2="5.969" y2="92.202" width="0.3048" layer="16"/>
 <wire x1="102.1588" y1="20.7382" x2="103.553" y2="20.7382" width="0.3048" layer="16"/>
-<wire x1="103.553" y1="20.7382" x2="103.58565" y2="20.77085" width="0.3048" layer="16" curve="90"/>
+<wire x1="103.553" y1="20.7382" x2="103.41565" y2="20.77085" width="0.3048" layer="16" curve="90"/>
 <wire x1="99.90865" y1="19.8247" x2="101.0158" y2="20.5747" width="0.3048" layer="16"/>
 <wire x1="101.0158" y1="20.5747" x2="102.0824" y2="20.5747" width="0.3048" layer="16"/>
 <wire x1="102.0824" y1="20.5747" x2="102.20235" y2="20.69465" width="0.3048" layer="16" curve="90"/>
-<wire x1="103.58565" y1="20.77085" x2="104.27335" y2="20.77085" width="0.3048" layer="16"/>
+<wire x1="103.41565" y1="20.77085" x2="104.27335" y2="20.77085" width="0.3048" layer="16"/>
 <wire x1="104.27335" y1="20.77085" x2="106.1466" y2="18.8976" width="0.3048" layer="16" curve="-90"/>
 <wire x1="106.1466" y1="18.8976" x2="108.08335" y2="16.96085" width="0.3048" layer="16" curve="90"/>
-<wire x1="108.08335" y1="16.96085" x2="108.74565" y2="16.96085" width="0.3048" layer="16"/>
+<wire x1="108.08335" y1="16.96085" x2="108.91565" y2="16.96085" width="0.3048" layer="16"/>
 <wire x1="111.7829" y1="18.89615" x2="111.7829" y2="17.2323" width="0.3048" layer="16"/>
 <wire x1="111.7829" y1="17.2323" x2="111.71465" y2="17.16405" width="0.3048" layer="16" curve="-90"/>
-<wire x1="108.74565" y1="16.96085" x2="109.3997" y2="16.3068" width="0.3048" layer="16" curve="90"/>
+<wire x1="108.91565" y1="16.96085" x2="109.3997" y2="16.3068" width="0.3048" layer="16" curve="90"/>
 <wire x1="109.3997" y1="16.3068" x2="111.252" y2="16.3068" width="0.3048" layer="16"/>
 <wire x1="111.252" y1="16.3068" x2="111.71465" y2="16.76945" width="0.3048" layer="16" curve="90"/>
@@
 <contactref element="U$63" pad="2"/>
 <contactref element="R13" pad="2"/>
-<wire x1="103.59835" y1="18.24355" x2="103.58565" y2="18.23085" width="0.3048" layer="16"/>
+<wire x1="103.59835" y1="18.24355" x2="103.41565" y2="18.23085" width="0.3048" layer="16"/>
 <wire x1="102.51985" y1="15.3924" x2="102.7938" y2="15.3924" width="0.3048" layer="16"/>
 <wire x1="102.7938" y1="15.3924" x2="104.3432" y2="16.9418" width="0.3048" layer="16" curve="90"/>
@@
 <via x="108.7374" y="17.6276" extent="1-16" drill="0.35"/>
 <wire x1="108.7374" y1="17.6276" x2="108.7374" y2="18.2226" width="0.3048" layer="16"/>
-<wire x1="108.7374" y1="18.2226" x2="108.74565" y2="18.23085" width="0.3048" layer="16" curve="-90"/>
+<wire x1="108.7374" y1="18.2226" x2="108.91565" y2="18.23085" width="0.3048" layer="16" curve="-90"/>
 </signal>
 <signal name="V_BATT">
@@
 <contactref element="J4" pad="1"/>
 <contactref element="R19" pad="1"/>
-<wire x1="108.74565" y1="20.77085" x2="110.5076" y2="20.77085" width="0.3048" layer="16"/>
+<wire x1="108.91565" y1="20.77085" x2="110.5076" y2="20.77085" width="0.3048" layer="16"/>
 <wire x1="110.5076" y1="20.77085" x2="110.8329" y2="21.09615" width="0.3048" layer="16" curve="90"/>
 <wire x1="107.48555" y1="7.7216" x2="107.3863875" y2="7.7216" width="0.3048" layer="16"/>
@@
 <via x="107.8484" y="20.7772" extent="1-16" drill="0.35"/>
 <wire x1="107.8484" y1="20.7772" x2="108.7393" y2="20.7772" width="0.3048" layer="16"/>
-<wire x1="108.7393" y1="20.7772" x2="108.74565" y2="20.77085" width="0.3048" layer="16" curve="-90"/>
+<wire x1="108.7393" y1="20.7772" x2="108.91565" y2="20.77085" width="0.3048" layer="16" curve="-90"/>
 <wire x1="110.8329" y1="21.09615" x2="111.60615" y2="21.8694" width="0.3048" layer="16" curve="-90"/>
 <wire x1="134.5438" y1="21.8694" x2="134.6454" y2="21.7678" width="0.3048" layer="16" curve="-90"/>
@@
 <contactref element="U$62" pad="C"/>
 <contactref element="U$62" pad="D"/>
-<wire x1="16.9898" y1="50.9914" x2="22.9898" y2="50.9914" width="0.3048" layer="16"/>
-<wire x1="16.9898" y1="50.9914" x2="16.9898" y2="49.4538" width="0.3048" layer="16"/>
+<wire x1="15.2898" y1="50.6164" x2="24.6898" y2="50.6164" width="0.3048" layer="16"/>
+<wire x1="15.2898" y1="50.6164" x2="16.9898" y2="49.4538" width="0.3048" layer="16"/>
 <wire x1="16.9898" y1="49.4538" x2="19.5298" y2="46.9138" width="0.3048" layer="16" curve="90"/>
 <wire x1="19.5298" y1="46.9138" x2="25.4762" y2="46.9138" width="0.3048" layer="16"/>

Commit message: updatyes
Parts:
- removed IC4: FS312F-G, FS312F-G:SOT95P280X145-6N
- removed Q4: FS8205, FS8205:FS8205
- removed R16: 2k, rcl:R0603
- added D62, D64, D65, D66, D67, D68, D69, D70, D71: 1N4148WS, Diodes:SOD-323
- added FUSE: 500m, rcl:R0603
- added IC1: XB3303ASOT23, Volume_V1:SOT23-3
- added J2: (no value), SparkFun-Connectors:1X04_NO_SILK
- added U$73, U$74: CHERRY-SOLDER, Volume_V1:CHERRY-SOLDER
- CN2: value (none) -> BM02B-SRSS-TB; device adafruit:JST-PH-2-SMT -> con-jst-sh:BM02B-SRSS-TB
- PROG1: device SparkFun-Connectors:1X06_HOLES_ONLY -> SparkFun-Connectors:1X06_NO_SILK
- U$14: device Volume_V1:CHERRY -> Volume_V1:CHERRY_CORNER_OFFED
- U$72: device Volume_V1:STAB-6U -> Volume_V1:STAB-6.25U
- moved LED2 78.9 mm to (179.8, 20.3), turned to 0 degrees
- moved CN2 73.0 mm to (143.9, 84.4), turned to 90 degrees
- moved J4 62.9 mm to (144.2, 80.1)
- moved IC3 35.6 mm to (89.1, 16.9)
- moved LED1 28.5 mm to (63.1, 19.1)
- moved R2 12.1 mm to (130.1, 10.7), turned to 270 degrees
- moved Q5 9.51 mm to (112.3, 10.6)
- moved R17 7.14 mm to (109.3, 10.2), turned to 90 degrees
- moved J1 4.95 mm to (67.3, 14.5)
- moved U$63 1.63 mm to (107.8, 19.0)
- moved C6 0.36 mm to (101.6, 9.73)
- moved R14 0.10 mm to (101.6, 17.4)
- moved C4 0.05 mm to (102.1, 19.9)
Connections:
- removed net N$77: IC4.1, Q4.4
- removed net N$78: IC4.3, Q4.6
- removed net N$79: C5.1, IC4.5, R15.1
- removed net N$80: IC4.2, R16.2
- new net N$68: D62.A, U$74.P$1
- new net N$69: C5.1, IC1.2, R15.1
- new net N$70: FUSE.2, J3.VBUS1, J3.VBUS2
- net COL14: now also U$73.P$2, U$74.P$2
- net D+: now also D64.A, J2.3
- net D-: now also D65.A, J2.2
- net GND: now also D64.C, D65.C, D66.C, D67.C, IC1.1, J2.4; no longer Q4.1, R16.1, U$68.P$1, U$68.P$2, U$68.P$3, U$68.P$4, U$68.P$5, U$68.P$6, U$68.P$7, U$68.P$8, U$69.P$1, U$69.P$2, U$69.P$3, U$69.P$4, U$69.P$5, U$69.P$6, U$69.P$7, U$69.P$8, U$70.P$1, U$70.P$2, U$70.P$3, U$70.P$4, U$70.P$5, U$70.P$6, U$70.P$7, U$70.P$8, U$71.P$1, U$71.P$2, U$71.P$3, U$71.P$4, U$71.P$5, U$71.P$6, U$71.P$7, U$71.P$8, U$72.P$1, U$72.P$2, U$72.P$3, U$72.P$4, U$72.P$5, U$72.P$6, U$72.P$7, U$72.P$8
- net G_BAT: now also CN2.1, IC1.3; no longer CN2.2, IC4.6, Q4.3
- net N$3: now also U$73.P$1
- net ROW3: now also D62.C
- net VDD_NRF: now also D66.A
- net V_BATT: now also CN2.2; no longer CN2.1
- net V_USB: now also D67.A, FUSE.1, J2.1; no longer J3.VBUS1, J3.VBUS2
Routing:
- net V_BATT: track 79.5 -> 169.3 mm, vias 4 -> 5
- net G_BAT: track 71.1 -> 156.9 mm, vias 2 -> 1
- net N$75: track 2.74 -> 86.6 mm, vias 0 -> 3
- net V_USB: track 238.7 -> 317.1 mm, vias 7 -> 11
- net ROW3: track 462.8 -> 522.6 mm, vias 0 -> 2
- net BLED: track 7.23 -> 46.2 mm
- net N$2: track 3.02 -> 34.4 mm
- net COL14: track 246.0 -> 268.3 mm, vias 4 -> 3
- net N$70: track 0.00 -> 19.9 mm, vias 0 -> 2
- net D+: track 211.8 -> 231.2 mm, vias 2 -> 7
- net D-: track 200.2 -> 218.9 mm, vias 2 -> 5
- net RESET: track 199.1 -> 217.6 mm
- net N$68: track 0.00 -> 13.0 mm, vias 0 -> 2
- net GND: track 28.1 -> 16.4 mm, vias 8 -> 5
- net N$81: track 21.7 -> 31.6 mm
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Other:
- board size 285.8 x 94.6 mm -> 283.5 x 94.6 mm
- board text added: "+"
- board text added: "D+"
- board text added: "D-"
- board text added: "POLARITY WORKS BT60"
- board text added: "SPARES"
- board text removed: "+ -"
- board text removed: "POLARITY WORKS 60"
