File: CRBN-60.sch (EAGLE design)
At the start: 160 parts, among them IC3 HOLYIOT_18010, IC4 FS312F-G, Q4 FS8205, Q5 PMOSFET, U2 AP2112K-3.3TRG1

Commit message: updatyes
Parts:
- removed IC4: FS312F-G, FS312F-G:FS312F-G
- removed Q4: FS8205, FS8205:FS8205
- removed R16: 2k, rcl:R-EU_R0603
- added D62, D64, D65, D66, D67, D68, D69, D70, D71: 1N4148WS, Diodes:1N4148WS
- added FUSE: 500m, rcl:R-EU_R0603
- added IC1: XB3303ASOT23, Volume_V1:XB3303ASOT23
- added J2: (no value), SparkFun-Connectors:CONN_041X04_NO_SILK
- added U$73, U$74: CHERRY-SOLDER, Volume_V1:CHERRY-SOLDER
- CN2: value (none) -> BM02B-SRSS-TB; device adafruit:JST_2PIN-SMT -> con-jst-sh:BM02B-SRSS-TB
- PROG1: device SparkFun-Connectors:CONN_06POGOPIN_HOLES_ONLY -> SparkFun-Connectors:CONN_06NO_SILK_FEMALE_PTH
- U$14: device Volume_V1:CHERRY -> Volume_V1:CHERRY_CORNER_OFFED
Connections:
- removed net N$77: IC4.OD, Q4.G2
- removed net N$78: IC4.OC, Q4.G1
- removed net N$79: C5.1, IC4.VCC, R15.1
- removed net N$80: IC4.CS, R16.2
- new net N$68: D62.A, U$74.2
- new net N$69: C5.1, IC1.VDD, R15.1
- new net N$70: FUSE.2, J3.VBUS
- net COL14: now also U$73.1, U$74.1
- net D+: now also D64.A, J2.3
- net D-: now also D65.A, J2.2
- net GND: now also D64.C, D65.C, D66.C, D67.C, IC1.VM, J2.4; no longer Q4.S1, R16.1, U$68.P$1, U$69.P$1, U$70.P$1, U$71.P$1, U$72.P$1
- net G_BAT: now also IC1.GND; no longer IC4.GND, Q4.S2
- net N$3: now also U$73.2
- net ROW3: now also D62.C
- net VDD_NRF: now also D66.A
- net V_USB: now also D67.A, FUSE.1, J2.1; no longer J3.VBUS
Other:
- moved on the sheet: C5, CN2
