File: BT60-soldered.brd (EAGLE design)
At the start: 283.8 x 94.6 mm, 214 parts, among them CN2 BM02B-SRSS-TB, IC3 HOLYIOT_18010, Q5 PMOSFET, U2 AP2112K-3.3TRG1, X5U_1 CHERRY-SOLDER, X5U_2 CHERRY-SOLDER

Commit message: further release tweaks
Parts:
- D69, D70, D71, D72: value 1N4148WS -> ESDSOD323; device Diodes:SOD-323 -> Volume_V1:SOD-323
