File: BT60-soldered.sch (EAGLE design)
At the start: 214 parts, among them CN2 BM02B-SRSS-TB, IC3 HOLYIOT_18010, Q5 PMOSFET, U2 AP2112K-3.3TRG1, X5U_1 CHERRY-SOLDER, X5U_2 CHERRY-SOLDER

Commit message: further release tweaks
Parts:
- D69, D70, D71, D72: value 1N4148WS -> ESDSOD323; device Diodes:1N4148WS -> Volume_V1:ESDSOD323
Changed lines of the file:
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@@
 <layer number="56" name="wert" color="7" fill="1" visible="no" active="no"/>
 <layer number="57" name="tCAD" color="7" fill="1" visible="no" active="no"/>
+<layer number="58" name="bCAD" color="7" fill="1" visible="no" active="no"/>
 <layer number="59" name="tCarbon" color="7" fill="1" visible="no" active="no"/>
 <layer number="60" name="bCarbon" color="7" fill="1" visible="no" active="no"/>
@@
 <layer number="154" name="FabDoc2" color="7" fill="1" visible="yes" active="yes"/>
 <layer number="155" name="FabDoc3" color="7" fill="1" visible="yes" active="yes"/>
+<layer number="166" name="AntennaArea" color="7" fill="1" visible="yes" active="yes"/>
+<layer number="168" name="4mmHeightArea" color="7" fill="1" visible="yes" active="yes"/>
 <layer number="191" name="mNets" color="7" fill="1" visible="yes" active="yes"/>
 <layer number="192" name="mBusses" color="7" fill="1" visible="yes" active="yes"/>
@@
 <part name="GND4" library="SparkFun-PowerSymbols" library_urn="urn:adsk.eagle:library:530" deviceset="GND" device=""/>
 <part name="SUPPLY1" library="SparkFun-PowerSymbols" library_urn="urn:adsk.eagle:library:530" deviceset="V_USB" device=""/>
-<part name="D69" library="Diodes" library_urn="urn:adsk.eagle:library:11396254" deviceset="1N4148WS" device="" package3d_urn="urn:adsk.eagle:package:10898396/3"/>
-<part name="D70" library="Diodes" library_urn="urn:adsk.eagle:library:11396254" deviceset="1N4148WS" device="" package3d_urn="urn:adsk.eagle:package:10898396/3"/>
-<part name="D71" library="Diodes" library_urn="urn:adsk.eagle:library:11396254" deviceset="1N4148WS" device="" package3d_urn="urn:adsk.eagle:package:10898396/3"/>
-<part name="D72" library="Diodes" library_urn="urn:adsk.eagle:library:11396254" deviceset="1N4148WS" device="" package3d_urn="urn:adsk.eagle:package:10898396/3"/>
+<part name="D69" library="Volume_V1" library_urn="urn:adsk.eagle:library:32198814" deviceset="ESDSOD323" device="" package3d_urn="urn:adsk.eagle:package:32198954/2"/>
+<part name="D70" library="Volume_V1" library_urn="urn:adsk.eagle:library:32198814" deviceset="ESDSOD323" device="" package3d_urn="urn:adsk.eagle:package:32198954/2"/>
+<part name="D71" library="Volume_V1" library_urn="urn:adsk.eagle:library:32198814" deviceset="ESDSOD323" device="" package3d_urn="urn:adsk.eagle:package:32198954/2"/>
+<part name="D72" library="Volume_V1" library_urn="urn:adsk.eagle:library:32198814" deviceset="ESDSOD323" device="" package3d_urn="urn:adsk.eagle:package:32198954/2"/>
 <part name="GND5" library="SparkFun-PowerSymbols" library_urn="urn:adsk.eagle:library:530" deviceset="GND" device=""/>
 <part name="SUPPLY2" library="SparkFun-PowerSymbols" library_urn="urn:adsk.eagle:library:530" deviceset="V_USB" device=""/>

Commit message: Update BT60-soldered.sch
Other:
- note added: "Battery Charging"
- note added: "Battery Connector"
- note added: "Battery Divider Power LED"
- note added: "Battery Protection"
- note added: "ESD Diodes Spares"
- note added: "Holyiot 18010"
- note added: "Pin Headers"
- note added: "Power Switching"
- note added: "Reset Button"
- note added: "Stabiliser and Screw Holes"
- note added: "USB Connector"
- moved on the sheet: C4, C5, C6, CN2, D63, D69, D70, D71, D72, D73, D74, D75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
